File: hardware/GsmBoard/GsmBoard.kicad_pcb (KiCad board)
At the start: 2 copper layers, 63.8 x 28.9 mm, 24 parts, among them J1 Power, J2 Serial, Q1 2N7002, Q2 2N7002, Q3 2N7002, U1 SIM800L-CORE, U2 LM2596S-ADJ

Commit message: main board power connector added to module
Parts:
- added J3: MainBoard Supply, Connector_JST:JST_XH_B2B-XH-A_1x02_P2.50mm_Vertical, F.Cu at (39.0, 194.2)
- moved C1 8.86 mm to (49.8, 194.2)
